File: pcbs/corne-chocolate/wireless/corne_choc_wireless/corne_choc_wireless.kicad_pcb (KiCad board)
At the start: 2 copper layers, 264 x 88.7 mm, 108 parts, among them J1 Conn_01x05, J2 Conn_01x02, J3 Conn_01x02, J4 Conn_01x05, SW1 Reset Button, SW2 SW_SPST, SW3 Reset Button, SW4 SW_SPST, U1 Nice_Nano_V2, U2 Nice_Nano_V2

Commit message: Gerber file V1
Gerber file V1
Parts:
- moved H13 86.8 mm to (153.9, 169.6)
- moved H7 86.8 mm to (143.0, 169.6)
- moved D41 86.4 mm to (196.3, 176.4)
- moved S40 86.4 mm to (166.4, 181.2)
- moved SW3 86.4 mm to (152.5, 150.1)
- moved SW4 86.4 mm to (152.5, 162.1)
- moved D23 86.4 mm to (207.0, 122.8)
- moved D40 86.4 mm to (169.8, 189.2)
- moved H11 86.4 mm to (222.5, 167.6)
- moved H8 86.4 mm to (261.5, 134.1)
- moved H9 86.4 mm to (261.5, 151.1)
- moved S22 86.4 mm to (180.5, 123.2)
- moved S23 86.4 mm to (198.5, 120.8)
- moved S24 86.4 mm to (216.5, 118.4)
- moved S25 86.4 mm to (234.5, 120.8)
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Routing:
- net r_row_0: track 116.9 -> 117.5 mm
- added copper zone on B.Cu, net (none)
- added copper zone on F.Cu, net (none)
Other:
- board size 264 x 88.7 mm -> 265 x 203.3 mm

Commit message: Gerber file V2
Gerber file V2
Parts:
- moved D13 1.00 mm to (35.0, 162.4)
- moved D14 1.00 mm to (53.0, 162.4)
- moved D15 1.00 mm to (71.0, 157.7)
- moved D16 1.00 mm to (89.0, 155.3)
- moved D17 1.00 mm to (107.0, 157.7)
- moved D18 1.00 mm to (125.0, 160.0)
- moved D19 1.00 mm to (98.0, 177.0)
- moved D20 1.00 mm to (117.1, 181.8)
- moved D21 1.00 mm to (137.0, 176.3)
- moved D34 1.00 mm to (189.0, 160.0)
- moved D35 1.00 mm to (207.0, 157.7)
- moved D36 1.00 mm to (225.0, 155.3)
- moved D37 1.00 mm to (243.0, 157.7)
- moved D38 1.00 mm to (261.0, 162.4)
- moved D39 1.00 mm to (279.0, 162.4)
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Routing:
- net r_col_4: track 110.3 -> 112.3 mm
- net r_col_3: track 127.6 -> 129.6 mm
- net r_col_2: track 122.1 -> 124.1 mm
- net col_4: track 100.6 -> 102.3 mm
- net col_5: track 87.3 -> 88.9 mm
- net r_col_5: track 88.7 -> 90.2 mm
- net col_3: track 117.9 -> 119.4 mm
- net Net-(D20-A): track 4.29 -> 5.76 mm
- net Net-(D41-A): track 4.29 -> 5.74 mm
- net r_row_3: track 112.5 -> 113.8 mm
- net col_1: track 131.3 -> 132.5 mm
- net col_0: track 148.6 -> 149.8 mm
- net col_2: track 112.1 -> 113.3 mm
- net r_col_0: track 166.7 -> 167.8 mm
- net r_row_2: track 136.9 -> 137.9 mm
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Other:
- outline, holes or cut-outs redrawn
